Commit message: wwwww

File: src/CXDL_ROS/cx_description/urdf/cx_description.urdf.xacro (robot description, xacro)
@@ -6,11 +6,14 @@
   name="cx_description"  xmlns:xacro="http://www.ros.org/wiki/xacro">
     <link
-  name="dummy">
+  name="world">
 </link>
 <joint
   name="dummy_joint"
   type="fixed">
+   <origin
+      xyz="0 0 2"
+      rpy="0 0 0" />
   <parent
-  link="dummy"/>
+  link="world"/>
   <child
   link="base_link"/>
